Commit message: refactoring(URDF file)

File: robots/megarover.urdf.xacro (robot description, xacro)
@@ -1,10 +1,10 @@
 <?xml version="1.0"?>
 <robot name="megarover20" xmlns:xacro="http://www.ros.org/wiki/xacro">
-	<xacro:include filename="$(find megarover_samples)/urdf/body/body.urdf.xacro"/>
-	<link name="base_footprint"/>
-	<xacro:body parent="base_footprint">
-		<origin xyz="0 0 0"/>
-	</xacro:body>
-	<material name="orange">
+  <xacro:include filename="$(find megarover_samples)/urdf/body/body.urdf.xacro"/>
+  <link name="base_footprint"/>
+  <xacro:body parent="base_footprint">
+    <origin xyz="0 0 0"/>
+  </xacro:body>
+  <material name="orange">
     <color rgba="1.0 0.5 0.2 1" />
   </material>
@@ -21,5 +21,5 @@
     </visual>
   </link>
-	<joint name="horizontal_laser_link_joint" type="fixed">
+  <joint name="horizontal_laser_link_joint" type="fixed">
     <parent link="base_link" />
     <child link="horizontal_laser_link" />

File: robots/vmegarover.urdf.xacro (robot description, xacro)
@@ -1,41 +1,41 @@
 <?xml version="1.0"?>
 <robot name="vmegarover" xmlns:xacro="http://www.ros.org/wiki/xacro">
-	<xacro:include filename="$(find megarover_samples)/urdf/body/vbody.urdf.xacro"/>
-	<xacro:include filename="$(find megarover_samples)/urdf/wheel/vwheel.urdf.xacro"/>
-	<xacro:include filename="$(find megarover_samples)/urdf/lrf/lrf.urdf.xacro"/>
+  <xacro:include filename="$(find megarover_samples)/urdf/body/vbody.urdf.xacro"/>
+  <xacro:include filename="$(find megarover_samples)/urdf/wheel/vwheel.urdf.xacro"/>
+  <xacro:include filename="$(find megarover_samples)/urdf/lrf/lrf.urdf.xacro"/>
   <!-- =============== Link & Joint =============== -->
   <!-- Base -->
   <link name="base_footprint"/>
   <xacro:base_v0 parent="base_footprint">
-	<origin xyz="0 0 0"/>
+    <origin xyz="0 0 0"/>
   </xacro:base_v0>
   <!-- Wheel -->
   <!-- Right Wheel -->
   <xacro:wheel_v0 prefix="right" parent="base_link">
-	<origin xyz="0 -0.14199 0.074742"/>
-	<axis xyz="0 1 0"/>
+    <origin xyz="0 -0.14199 0.074742"/>
+    <axis xyz="0 1 0"/>
   </xacro:wheel_v0>
   <!-- Left Wheel -->
   <xacro:wheel_v0 prefix="left" parent="base_link">
-	<origin xyz="0 0.14199 0.074742"  rpy="0 0 ${M_PI}" />
-	<axis xyz="0 -1 0"/>
+    <origin xyz="0 0.14199 0.074742"  rpy="0 0 ${M_PI}" />
+    <axis xyz="0 -1 0"/>
   </xacro:wheel_v0>
   <!-- Front LRF -->
   <xacro:lrf_v0 prefix="front" parent="base_link">
-  	<origin xyz="0.099 0 0.1015"/>
+    <origin xyz="0.099 0 0.1015"/>
   </xacro:lrf_v0>
   <!-- Front LRF Upper-->
   <!-- <xacro:lrf_v0 prefix="front" parent="base_link">
-  	<origin xyz="0.099 0 0.2155"  rpy="${M_PI} 0 0" />
+    <origin xyz="0.099 0 0.2155"  rpy="${M_PI} 0 0" />
   </xacro:lrf_v0> -->
   <!-- Rear LRF -->
   <!-- xacro:lrf_v0 prefix="rear" parent="base_link">
-  	<origin xyz="-0.289 0 0.1015"  rpy="0 0 ${M_PI}" />
+    <origin xyz="-0.289 0 0.1015"  rpy="0 0 ${M_PI}" />
   </xacro:lrf_v0 -->
   <link name="lrf_link"/>
   <joint name="lrf_link_joint" type="fixed">
-	<parent link="base_footprint"/>
-	<child link="lrf_link"/>
-	<origin xyz="0.099 0 0.1015"/>
+    <parent link="base_footprint"/>
+    <child link="lrf_link"/>
+    <origin xyz="0.099 0 0.1015"/>
   </joint>
   <!-- ===============  Transmission =============== -->
@@ -55,8 +55,8 @@
   <!-- LRF -->
   <xacro:lrf_gazebo_v0 prefix="front"
-					   min_rad="-1.57" max_rad="1.57"
-					   min_range="0.06" max_range="4.0"/>
+                       min_rad="-1.57" max_rad="1.57"
+                       min_range="0.06" max_range="4.0"/>
   <!-- xacro:lrf_gazebo_v0 prefix="rear"
-					   min_rad="-1.57" max_rad="1.57"
-					   min_range="0.06" max_range="4.0"/ -->
+                       min_rad="-1.57" max_rad="1.57"
+                       min_range="0.06" max_range="4.0"/ -->
 </robot>

File: urdf/body/body.urdf.xacro (robot description, xacro)
@@ -1,20 +1,20 @@
 <?xml version="1.0"?>
 <robot xmlns:xacro="http://www.ros.org/wiki/xacro">
-	<xacro:macro name="body" params="parent *joint_origin">
-		<joint name="base_joint" type="fixed">
-			<xacro:insert_block name="joint_origin"/>
-			<parent link="${parent}"/>
-			<child  link="base_link"/>
-		</joint>
-		<link name="base_link">
-			<visual>
-				<origin xyz="-0.028241 -0.073553 0.01"/>
-				<geometry>
-					<mesh filename="package://megarover_samples/meshes/dae/megarover.dae"/>
-					<!--<mesh filename="$(find kobuki_description)/meshes/main_body.dae"/>-->
-					<!--<mesh filename="/home/rover/3d/megarover.dae"/>-->
-				</geometry>
-			</visual>
-		</link>
-	</xacro:macro>
+  <xacro:macro name="body" params="parent *joint_origin">
+    <joint name="base_joint" type="fixed">
+      <xacro:insert_block name="joint_origin"/>
+      <parent link="${parent}"/>
+      <child  link="base_link"/>
+    </joint>
+    <link name="base_link">
+      <visual>
+        <origin xyz="-0.028241 -0.073553 0.01"/>
+        <geometry>
+          <mesh filename="package://megarover_samples/meshes/dae/megarover.dae"/>
+          <!--<mesh filename="$(find kobuki_description)/meshes/main_body.dae"/>-->
+          <!--<mesh filename="/home/rover/3d/megarover.dae"/>-->
+        </geometry>
+      </visual>
+    </link>
+  </xacro:macro>
 </robot>

File: urdf/body/vbody.urdf.xacro (robot description, xacro)
@@ -3,28 +3,28 @@
   <xacro:include filename="$(find megarover_samples)/urdf/body/body.gazebo.xacro"/>
   <xacro:macro name="base_v0" params="parent *joint_origin">
-	<joint name="base_link_joint" type="fixed">
-	  <insert_block name="joint_origin"/>
-	  <parent link="${parent}"/>
-	  <child link="base_link"/>
-	</joint>
-	<link name="base_link">
-	  <visual>
-		<geometry>
-		  <mesh filename="package://megarover_samples/meshes/dae/vmega_body.dae"/>
-		</geometry>
-	  </visual>
-	  <collision>
-		<geometry>
-		  <mesh filename="package://megarover_samples/meshes/stl/vmega_body.stl"/>
-		</geometry>
-	  </collision>
-	  <inertial>
-		<origin xyz="-0.061 0 -0.002"/>
-		<mass value="13.754"/>
-		<inertia ixx="0.110655982" ixy="0" ixz="0"
-				 iyy="0.20062619" iyz="0"
-				 izz="0.269504336" />
-	  </inertial>
-	</link>
+    <joint name="base_link_joint" type="fixed">
+      <insert_block name="joint_origin"/>
+      <parent link="${parent}"/>
+      <child link="base_link"/>
+    </joint>
+    <link name="base_link">
+      <visual>
+        <geometry>
+          <mesh filename="package://megarover_samples/meshes/dae/vmega_body.dae"/>
+        </geometry>
+      </visual>
+      <collision>
+        <geometry>
+          <mesh filename="package://megarover_samples/meshes/stl/vmega_body.stl"/>
+        </geometry>
+      </collision>
+      <inertial>
+        <origin xyz="-0.061 0 -0.002"/>
+        <mass value="13.754"/>
+        <inertia ixx="0.110655982" ixy="0" ixz="0"
+          iyy="0.20062619" iyz="0"
+          izz="0.269504336" />
+      </inertial>
+    </link>
   </xacro:macro>
 </robot>

File: urdf/common.xacro (robot description, xacro)
@@ -3,14 +3,14 @@
   <property name="M_PI" value="3.14159274"/>
   <xacro:macro name="cylinder_inertial" params="mass radius length">
-	<mass value="${mass}"/>
-	<inertia ixx="${((radius*radius)/4 + (length*length)/12)*mass}" ixy="0" ixz="0"
-			 iyy="${((radius*radius)/4 + (length*length)/12)*mass}" iyz="0"
-			 izz="${(mass*radius*radius)/2}" />
+    <mass value="${mass}"/>
+    <inertia ixx="${((radius*radius)/4 + (length*length)/12)*mass}" ixy="0" ixz="0"
+      iyy="${((radius*radius)/4 + (length*length)/12)*mass}" iyz="0"
+      izz="${(mass*radius*radius)/2}" />
   </xacro:macro>
   <xacro:macro name="box_inertial" params="mass height width depth">
-	<mass value="${mass}"/>
-	<inertia ixx="${(mass*(width*width+depth*depth))/12}" ixy="0" ixz="0"
-			 iyy="${(mass*(height*height+depth*depth))/12}" iyz="0"
-			 izz="${(mass*(height*height+width*width))/12}" />
+    <mass value="${mass}"/>
+    <inertia ixx="${(mass*(width*width+depth*depth))/12}" ixy="0" ixz="0"
+      iyy="${(mass*(height*height+depth*depth))/12}" iyz="0"
+      izz="${(mass*(height*height+width*width))/12}" />
   </xacro:macro>
 </robot>

File: urdf/lrf/lrf.urdf.xacro (robot description, xacro)
@@ -4,25 +4,25 @@
   <xacro:include filename="$(find megarover_samples)/urdf/lrf/lrf.gazebo.xacro"/>
   <xacro:macro name="lrf_v0" params="prefix parent *joint_origin">
-		<joint name="${prefix}_lrf_joint" type="fixed">
-			<insert_block name="joint_origin"/>
-			<parent link="${parent}"/>
-			<child link="${prefix}_lrf_link"/>
-		</joint>
-		<link name="${prefix}_lrf_link">
-			<visual>
-			<geometry>
-				<mesh filename="package://megarover_samples/meshes/dae/lrf.dae"/>
-			</geometry>
-			</visual>
-			<collision>
-				<geometry>
-					<mesh filename="package://megarover_samples/meshes/stl/lrf.stl"/>
-				</geometry>
-			</collision>
-			<inertial>
-				<origin xyz="0 0 0"/>
-				<box_inertial mass="0.218" height="0.07" width="0.05" depth="0.05"/>
-			</inertial>
-		</link>
+    <joint name="${prefix}_lrf_joint" type="fixed">
+      <insert_block name="joint_origin"/>
+      <parent link="${parent}"/>
+      <child link="${prefix}_lrf_link"/>
+    </joint>
+    <link name="${prefix}_lrf_link">
+      <visual>
+        <geometry>
+          <mesh filename="package://megarover_samples/meshes/dae/lrf.dae"/>
+        </geometry>
+      </visual>
+      <collision>
+        <geometry>
+          <mesh filename="package://megarover_samples/meshes/stl/lrf.stl"/>
+        </geometry>
+      </collision>
+      <inertial>
+        <origin xyz="0 0 0"/>
+        <box_inertial mass="0.218" height="0.07" width="0.05" depth="0.05"/>
+      </inertial>
+    </link>
   </xacro:macro>
 </robot>

File: urdf/wheel/vwheel.urdf.xacro (robot description, xacro)
@@ -8,28 +8,28 @@
   <property name="wheel_mass" value="0.823"/>
   <xacro:macro name="wheel_v0" params="prefix parent *joint_origin *joint_axis">
-		<joint name="${prefix}_wheel_joint" type="continuous">
-			<insert_block name="joint_origin"/>
-			<parent link="${parent}"/>
-			<child link="${prefix}_wheel_link"/>
-			<insert_block name="joint_axis"/>
-		</joint>
-		<link name="${prefix}_wheel_link">
-			<visual>
-			<geometry>
-				<mesh filename="package://megarover_samples/meshes/dae/vmega_wheel.dae"/>
-			</geometry>
-			</visual>
-			<collision>
-				<origin xyz="0 0 0" rpy="${-M_PI/2} 0 0"/>
-				<geometry>
-					<cylinder radius="${wheel_radius}" length="${wheel_length}"/>
-				</geometry>
-			</collision>
-			<inertial>
-				<origin xyz="0 0 0" rpy="${-M_PI/2} 0 0"/>
-				<cylinder_inertial mass="${wheel_mass}"
-									 radius="${wheel_radius}" length="${wheel_length}"/>
-			</inertial>
-		</link>
+    <joint name="${prefix}_wheel_joint" type="continuous">
+      <insert_block name="joint_origin"/>
+      <parent link="${parent}"/>
+      <child link="${prefix}_wheel_link"/>
+      <insert_block name="joint_axis"/>
+    </joint>
+    <link name="${prefix}_wheel_link">
+      <visual>
+        <geometry>
+          <mesh filename="package://megarover_samples/meshes/dae/vmega_wheel.dae"/>
+        </geometry>
+      </visual>
+      <collision>
+        <origin xyz="0 0 0" rpy="${-M_PI/2} 0 0"/>
+        <geometry>
+          <cylinder radius="${wheel_radius}" length="${wheel_length}"/>
+        </geometry>
+      </collision>
+      <inertial>
+        <origin xyz="0 0 0" rpy="${-M_PI/2} 0 0"/>
+        <cylinder_inertial mass="${wheel_mass}"
+          radius="${wheel_radius}" length="${wheel_length}"/>
+      </inertial>
+    </link>
   </xacro:macro>
 </robot>

File: urdf/wheel/wheel.transmission.xacro (robot description, xacro)
@@ -2,14 +2,14 @@
 <robot xmlns:xacro="http://ros.org/wiki/xacro">
   <xacro:macro name="wheel_trans_v0" params="prefix">
-	<transmission name="${prefix}_wheel_trans">
+    <transmission name="${prefix}_wheel_trans">
       <type>transmission_interface/SimpleTransmission</type>
       <joint name="${prefix}_wheel_joint">
-		<hardwareInterface>VelocityJointInterface</hardwareInterface>
+        <hardwareInterface>VelocityJointInterface</hardwareInterface>
       </joint>
-	  <actuator name="${prefix}_wheel_motor">
-		<hardwareInterface>VelocityJointInterface</hardwareInterface>
-		<mechanicalReduction>30</mechanicalReduction>
+      <actuator name="${prefix}_wheel_motor">
+        <hardwareInterface>VelocityJointInterface</hardwareInterface>
+        <mechanicalReduction>30</mechanicalReduction>
       </actuator>
-	</transmission>
+    </transmission>
   </xacro:macro>
 </robot>
