Commit message: インデントの修正

File: urdf/wheel/wheel.transmission.xacro (robot description, xacro)
@@ -3,12 +3,12 @@
   <xacro:macro name="wheel_trans_v0" params="prefix">
 	<transmission name="${prefix}_wheel_trans">
-      <type>transmission_interface/SimpleTransmission</type>
-      <joint name="${prefix}_wheel_joint">
-		<hardwareInterface>hardware_interface/VelocityJointInterface</hardwareInterface>
-      </joint>
+    <type>transmission_interface/SimpleTransmission</type>
+    <joint name="${prefix}_wheel_joint">
+      <hardwareInterface>hardware_interface/VelocityJointInterface</hardwareInterface>
+    </joint>
 	  <actuator name="${prefix}_wheel_motor">
-		<hardwareInterface>hardware_interface/VelocityJointInterface</hardwareInterface>
-		<mechanicalReduction>30</mechanicalReduction>
-      </actuator>
+      <hardwareInterface>hardware_interface/VelocityJointInterface</hardwareInterface>
+      <mechanicalReduction>30</mechanicalReduction>
+    </actuator>
 	</transmission>
   </xacro:macro>
