Commit message: イナーシャの修正、ファイル名に空白が入っていた点を修正

File: urdf/body/vbody.urdf.xacro (robot description, xacro)
@@ -22,7 +22,7 @@
 		<origin xyz="-0.061 0 -0.002"/>
 		<mass value="13.754"/>
-		<inertia ixx="1.64890" ixy="0" ixz="-0.21424"
-				 iyy="2.24766" iyz="0"
-				 izz="1.25664" />
+		<inertia ixx="0.110655982" ixy="0" ixz="0"
+				 iyy="0.20062619" iyz="0"
+				 izz="0.269504336" />
 	  </inertial>
 	</link>

Commit message: add xacro namespace

File: urdf/body/vbody.urdf.xacro (robot description, xacro)
@@ -4,5 +4,5 @@
   <xacro:macro name="base_v0" params="parent *joint_origin">
     <joint name="base_link_joint" type="fixed">
-      <insert_block name="joint_origin"/>
+      <xacro:insert_block name="joint_origin"/>
       <parent link="${parent}"/>
       <child link="base_link"/>

File: urdf/common.xacro (robot description, xacro)
@@ -1,5 +1,5 @@
 <?xml version="1.0"?>
 <robot xmlns:xacro="http://ros.org/wiki/xacro">
-  <property name="M_PI" value="3.14159274"/>
+  <xacro:property name="M_PI" value="3.14159274"/>
   <xacro:macro name="cylinder_inertial" params="mass radius length">
     <mass value="${mass}"/>

File: urdf/lrf/lrf.urdf.xacro (robot description, xacro)
@@ -5,5 +5,5 @@
   <xacro:macro name="lrf_v0" params="prefix parent *joint_origin">
     <joint name="${prefix}_lrf_joint" type="fixed">
-      <insert_block name="joint_origin"/>
+      <xacro:insert_block name="joint_origin"/>
       <parent link="${parent}"/>
       <child link="${prefix}_lrf_link"/>
@@ -22,5 +22,5 @@
       <inertial>
         <origin xyz="0 0 0"/>
-        <box_inertial mass="0.218" height="0.07" width="0.05" depth="0.05"/>
+        <xacro:box_inertial mass="0.218" height="0.07" width="0.05" depth="0.05"/>
       </inertial>
     </link>

File: urdf/wheel/vwheel.urdf.xacro (robot description, xacro)
@@ -4,13 +4,13 @@
   <xacro:include filename="$(find megarover_samples)/urdf/wheel/wheel.transmission.xacro"/>
   <xacro:include filename="$(find megarover_samples)/urdf/wheel/wheel.gazebo.xacro"/>
-  <property name="wheel_radius" value="0.076"/>
-  <property name="wheel_length" value="0.03"/>
-  <property name="wheel_mass" value="0.823"/>
+  <xacro:property name="wheel_radius" value="0.076"/>
+  <xacro:property name="wheel_length" value="0.03"/>
+  <xacro:property name="wheel_mass" value="0.823"/>
   <xacro:macro name="wheel_v0" params="prefix parent *joint_origin *joint_axis">
     <joint name="${prefix}_wheel_joint" type="continuous">
-      <insert_block name="joint_origin"/>
+      <xacro:insert_block name="joint_origin"/>
       <parent link="${parent}"/>
       <child link="${prefix}_wheel_link"/>
-      <insert_block name="joint_axis"/>
+      <xacro:insert_block name="joint_axis"/>
     </joint>
     <link name="${prefix}_wheel_link">
@@ -28,5 +28,5 @@
       <inertial>
         <origin xyz="0 0 0" rpy="${-M_PI/2} 0 0"/>
-        <cylinder_inertial mass="${wheel_mass}"
+        <xacro:cylinder_inertial mass="${wheel_mass}"
           radius="${wheel_radius}" length="${wheel_length}"/>
       </inertial>
